Commit message: changes trying to fix slam

File: rr_ws/src/rr_description/urdf/RogueRover.urdf (robot description, URDF)
Before this commit: robot RogueRover, 17 links, 16 joints
Links:
- removed link arm_link1
- removed link arm_link2
- removed link arm_link3
- removed link arm_link4
- removed link arm_link5
- removed link llink1
- removed link llink2
- removed link llink3
- removed link mono_link
- removed link rlink1
- removed link rlink2
- removed link rlink3
- added link back_left_wheel, mass 0.0515309299357028; collision mesh filename=package://rr_description/meshes/back_left_wheel_X3.STL; visual mesh filename=package://rr_description/meshes/back_left_wheel_X3.STL
- added link back_right_wheel, mass 0.051540174053366; collision mesh filename=package://rr_description/meshes/back_right_wheel_X3.STL; visual mesh filename=package://rr_description/meshes/back_right_wheel_X3.STL
- added link front_left_wheel, mass 0.051543; collision mesh filename=package://rr_description/meshes/front_left_wheel_X3.STL; visual mesh filename=package://rr_description/meshes/front_left_wheel_X3.STL
- added link front_right_wheel, mass 0.051532; collision mesh filename=package://rr_description/meshes/front_right_wheel_X3.STL; visual mesh filename=package://rr_description/meshes/front_right_wheel_X3.STL
- link base_link: mass 1.0754239466482 -> 0.486218814966626; geometry collision mesh filename=package://rr_description/meshes/base_link_X3.STL; visual mesh filename=package://rr_description/meshes/base_link_X3.STL
- link camera_link: mass 0.224346273348015 -> 0; geometry collision mesh filename=package://rr_description/meshes/camera_link.STL; visual mesh filename=package://rr_description/meshes/camera_link.STL
- link laser_link: mass 0.0433399617554554 -> 0.0483909504209895; geometry collision mesh filename=package://rr_description/meshes/laser_link.STL; visual mesh filename=package://rr_description/meshes/laser_link.STL
Joints:
- removed joint arm_joint1
- removed joint arm_joint2
- removed joint arm_joint3
- removed joint arm_joint4
- removed joint arm_joint5
- removed joint astra_joint
- removed joint grip_joint
- removed joint llink_joint1
- removed joint llink_joint2
- removed joint llink_joint3
- removed joint mono_joint
- removed joint rlink_joint2
- removed joint rlink_joint3
- added joint back_left_joint: type continuous, parent base_link, child back_left_wheel, origin xyz=-0.08 0.084492 -0.03954 rpy=1.5703 0 0, axis 0 0 1, limit effort=100 velocity=1
- added joint back_right_joint: type continuous, parent base_link, child back_right_wheel, origin xyz=-0.08 -0.0845 -0.03946 rpy=-1.57 0 3.14159, axis 0 0 1, limit effort=100 velocity=1
- added joint camera_joint: type fixed, parent base_link, child camera_link, origin xyz=0.057105 1.7948E-05 0.03755 rpy=0 0 0
- added joint front_left_joint: type continuous, parent base_link, child front_left_wheel, origin xyz=0.08 0.084492 -0.0389 rpy=1.5703 0 0, axis 0 0 1, limit effort=100 velocity=1
- added joint front_right_joint: type continuous, parent base_link, child front_right_wheel, origin xyz=0.08 -0.0845 -0.0389 rpy=-1.5703 0 3.14159, axis 0 0 1, limit effort=100 velocity=1
- joint base_imu: origin xyz=0.001 0.017 0.0322 rpy=0 3.1415 1.5707 -> xyz=-0.06 0.01 0.01 rpy=0 3.1415 1.5707
- joint base_joint: origin xyz=0.0 0.0 0.076 rpy=0 0 0 -> xyz=0.0 0.0 0.0815 rpy=0 0 0
- joint laser_joint: origin xyz=0.10478 0 0.0471 rpy=0 0 0 -> xyz=0.0435 5.25826986680105E-05 0.11 rpy=0 0 0
